File: Pogo_pcb/Pogo_pcb.kicad_sch (KiCad schematic)
At the start: 0 parts

Commit message: Pogo PCB
Parts:
- added C1, C7: 1uF, Capacitor_SMD:C_0805_2012Metric_Pad1.18x1.45mm_HandSolder, symbol Device:C
- added D1: LED, LED_SMD:LED_0402_1005Metric_Pad0.77x0.64mm_HandSolder, symbol Device:LED
- added D2, D3, D4: SS14, Diode_SMD:D_SMA, symbol Diode:SS14
- added IC2: ADPL40502AUJZ-3.0-R7, Package_TO_SOT_SMD:SOT-23-5_HandSoldering, symbol ADPL40502AUJZ-3_0-R7:ADPL40502AUJZ-3.0-R7
- added J1, J2: Conn_01x02_Pin, Connector_PinSocket_2.54mm:PinSocket_1x02_P2.54mm_Vertical, symbol Connector:Conn_01x02_Pin
- added R1: 330, Resistor_SMD:R_0402_1005Metric_Pad0.72x0.64mm_HandSolder, symbol Device:R
- added R2: 15k, Resistor_SMD:R_0402_1005Metric_Pad0.72x0.64mm_HandSolder, symbol Device:R
- added U1: ~, Pogo_pin:Pogo_pin, symbol Pogo_library:Pogo_male
- added U2: LTC4054XES5-4.2, Package_TO_SOT_SMD:TSOT-23-5_HandSoldering, symbol Battery_Management:LTC4054XES5-4.2
Connections:
- new net: D1.1 (K), U2.1 (~{CHRG})
- new net: D1.2 (A), R1.2
- new net: D2.2 (A), U1.1, U1.3
- new net: R2.1, U2.5 (PROG)
- new net: C7.2, D3.1 (K), D4.1 (K), IC2.1 (VIN), IC2.3 (EN)
- new net +5V: C1.2, D2.1 (K), D3.2 (A), R1.1, U2.4 (V_{CC})
- new net GND: C1.1, C7.1, IC2.2 (GND), J1.2 (Pin_2), J2.2 (Pin_2), R2.2, U1.2, U2.2 (GND)
- new net VBUS: D4.2 (A), J1.1 (Pin_1), U2.3 (BAT)
- new net VDD: IC2.5 (VOUT), J2.1 (Pin_1)
Other:
- note added: "Battery Pins"
- note added: "Charger"
- note added: "For 10mA"
- note added: "Or 1.5k for 100mA"
- note added: "Output Pins"
- note added: "Pogo Pin Connector"
- note added: "Voltage Regulator"
