File: Pogo_pcb/Pogo_pcb.kicad_pcb (KiCad board)
At the start: 2 copper layers, 20.6 x 22 mm, 13 parts, among them IC2 ADPL40502AUJZ-3.0-R7, J1 Conn_01x02_Pin, J2 Conn_01x02_Pin, U2 LTC4054XES5-4.2

Commit message: Small Wireless
Parts:
- C1, C7: footprint Capacitor_SMD:C_0805_2012Metric_Pad1.18x1.45mm_HandSolder -> Capacitor_SMD:C_0402_1005Metric_Pad0.74x0.62mm_HandSolder
- moved C1 0.84 mm to (152.9, 60.8)
- moved C7 0.49 mm to (150.4, 60.2)
Routing:
- net GND: track 10.2 -> 8.05 mm
- net +5V: track 18.4 -> 20.1 mm
- net Net-(D3-K): track 17.2 -> 18.3 mm
